Commit message: Add dual arm controllers and launch configuration for agilex_piper

File: piper_bringup/urdf/agilex_piper_dual.system.xacro (robot description, xacro)
@@ -7,16 +7,26 @@
   <xacro:arg name="sim_isaac_sim" default="false"/>
   <xacro:arg name="simulation_controllers" default=""/>
-  <xacro:arg name="prefix" default=""/>
   <!-- Define base_link -->
   <link name="base_link"/>
   <!-- Include the urdf macro -->
   <xacro:include filename="$(find piper_bringup)/urdf/agilex_piper_macro.urdf.xacro"/>
-  <xacro:agilex_piper name="agilex_piper" parent="base_link" prefix="$(arg prefix)">
-    <origin xyz="0 0 0" rpy="0 0 0" />
+  <xacro:agilex_piper name="arm" parent="base_link" prefix="left_">
+    <origin xyz="-0.35 0 0" rpy="0 0 0" />
+  </xacro:agilex_piper>
+  <xacro:agilex_piper name="arm" parent="base_link" prefix="right_">
+    <origin xyz="0.35 0 0" rpy="0 0 0" />
   </xacro:agilex_piper>
   <!-- Include the ros2_control macro -->
   <xacro:include filename="$(find piper_bringup)/urdf/agilex_piper_macro.ros2_control.xacro"/>
-  <xacro:agilex_piper_ros2_control  name="agilex_piper_ros2_control"
-                                    prefix="$(arg prefix)"
+  <xacro:agilex_piper_ros2_control  name="left_arm_ros2_control"
+                                    prefix="left_"
+                                    use_mock_hardware="$(arg use_mock_hardware)"
+                                    mock_sensor_commands="$(arg mock_sensor_commands)"
+                                    sim_gazebo_classic="$(arg sim_gazebo_classic)"
+                                    sim_gazebo="$(arg sim_gazebo)"
+                                    sim_isaac_sim="$(arg sim_isaac_sim)"
+                                    simulation_controllers="$(arg simulation_controllers)"/>
+  <xacro:agilex_piper_ros2_control  name="right_arm_ros2_control"
+                                    prefix="right_"
                                     use_mock_hardware="$(arg use_mock_hardware)"
                                     mock_sensor_commands="$(arg mock_sensor_commands)"

File: piper_bringup/urdf/agilex_piper_macro.ros2_control.xacro (robot description, xacro)
@@ -3,4 +3,5 @@
   <xacro:macro name="agilex_piper_ros2_control" params="
                name
+               prefix:=''
                use_mock_hardware:=false
                mock_sensor_commands:=false

File: piper_bringup/urdf/agilex_piper_macro.urdf.xacro (robot description, xacro)
@@ -1,8 +1,8 @@
 <?xml version="1.0"?>
 <robot name="agilex_piper" xmlns:xacro="http://www.ros.org/wiki/xacro">
-  <xacro:macro name="agilex_piper" params="*origin name=agilex_piper parent=base_link">
+  <xacro:macro name="agilex_piper" params="*origin name=agilex_piper parent=base_link prefix=''">
     <!-- agilex_piper's root link -->
-    <xacro:property name="root_link" value="${name}"/>
-    <joint name="${name}_joint" type="fixed">
+    <xacro:property name="root_link" value="${prefix}${name}"/>
+    <joint name="${prefix}${name}_joint" type="fixed">
       <xacro:insert_block name="origin"/>
         <parent link="${parent}"/>
@@ -31,5 +31,5 @@
       </collision>
     </link>
-    <link name="link1">
+    <link name="${prefix}link1">
       <inertial>
         <origin xyz="0.00032 -0.00041 -0.00348" rpy="0 0 0" />
@@ -53,12 +53,12 @@
       </collision>
     </link>
-    <joint name="joint1" type="revolute">
+    <joint name="${prefix}joint1" type="revolute">
       <origin xyz="0 0 0.123" rpy="0 0 0" />
       <parent link="${root_link}" />
-      <child link="link1" />
+      <child link="${prefix}link1" />
       <axis xyz="0 0 1" />
       <limit lower="-2.618" upper="2.618" effort="100" velocity="5" />
     </joint>
-    <link name="link2">
+    <link name="${prefix}link2">
       <inertial>
         <origin xyz="0.21852 -0.00861 0.00126" rpy="0 0 0" />
@@ -82,12 +82,12 @@
       </collision>
     </link>
-    <joint name="joint2" type="revolute">
+    <joint name="${prefix}joint2" type="revolute">
       <origin xyz="0 0 0" rpy="1.5708 -0.10095 -3.1416" />
-      <parent link="link1" />
-      <child link="link2" />
+      <parent link="${prefix}link1" />
+      <child link="${prefix}link2" />
       <axis xyz="0 0 1" />
       <limit lower="0" upper="3.14" effort="100" velocity="5" />
     </joint>
-    <link name="link3">
+    <link name="${prefix}link3">
       <inertial>
         <origin xyz="-0.01999 -0.14808 -0.00053" rpy="0 0 0" />
@@ -111,12 +111,12 @@
       </collision>
     </link>
-    <joint name="joint3" type="revolute">
+    <joint name="${prefix}joint3" type="revolute">
       <origin xyz="0.28503 0 0" rpy="0 0 -1.759" />
-      <parent link="link2" />
-      <child link="link3" />
+      <parent link="${prefix}link2" />
+      <child link="${prefix}link3" />
       <axis xyz="0 0 1" />
       <limit lower="-2.967" upper="0" effort="100" velocity="5" />
     </joint>
-    <link name="link4">
+    <link name="${prefix}link4">
       <inertial>
         <origin xyz="0.00013 -0.00076 -0.00394" rpy="0 0 0" />
@@ -140,12 +140,12 @@
       </collision>
     </link>
-    <joint name="joint4" type="revolute">
+    <joint name="${prefix}joint4" type="revolute">
       <origin xyz="-0.021984 -0.25075 0" rpy="1.5708 0 0" />
-      <parent link="link3" />
-      <child link="link4" />
+      <parent link="${prefix}link3" />
+      <child link="${prefix}link4" />
       <axis xyz="0 0 1" />
       <limit lower="-1.745" upper="1.745" effort="100" velocity="5" />
     </joint>
-    <link name="link5">
+    <link name="${prefix}link5">
       <inertial>
         <origin xyz="0.00018 -0.06104 -0.00227" rpy="0 0 0" />
@@ -169,12 +169,12 @@
       </collision>
     </link>
-    <joint name="joint5" type="revolute">
+    <joint name="${prefix}joint5" type="revolute">
       <origin xyz="0 0 0" rpy="-1.5708 0 0" />
-      <parent link="link4" />
-      <child link="link5" />
+      <parent link="${prefix}link4" />
+      <child link="${prefix}link5" />
       <axis xyz="0 0 1" />
       <limit lower="-1.22" upper="1.22" effort="100" velocity="5" />
     </joint>
-    <link name="link6">
+    <link name="${prefix}link6">
       <inertial>
         <origin xyz="-0.00003 0.00006 0.04618" rpy="0 0 0" />
@@ -198,8 +198,8 @@
       </collision>
     </link>
-    <joint name="joint6" type="revolute">
+    <joint name="${prefix}joint6" type="revolute">
       <origin xyz="8.8259E-05 -0.091 0" rpy="1.5708 0 0" />
-      <parent link="link5" />
-      <child link="link6" />
+      <parent link="${prefix}link5" />
+      <child link="${prefix}link6" />
       <axis xyz="0 0 1" />
       <limit lower="-2.0944" upper="2.0944" effort="100" velocity="5" />

File: piper_bringup/urdf/include/isaac_sim.ros2_control.xacro (robot description, xacro)
@@ -8,5 +8,5 @@
           <param name="trigger_joint_command_threshold">-1.0</param>
     </hardware>
-    <joint name="joint1">
+    <joint name="${prefix}joint1">
         <command_interface name="position"/>
         <state_interface name="position">
@@ -16,5 +16,5 @@
         <state_interface name="effort"/>
     </joint>
-    <joint name="joint2">
+    <joint name="${prefix}joint2">
         <command_interface name="position"/>
         <state_interface name="position">
@@ -24,5 +24,5 @@
         <state_interface name="effort"/>
     </joint>
-    <joint name="joint3">
+    <joint name="${prefix}joint3">
         <command_interface name="position"/>
         <state_interface name="position">
@@ -32,5 +32,5 @@
         <state_interface name="effort"/>
     </joint>
-    <joint name="joint4">
+    <joint name="${prefix}joint4">
         <command_interface name="position"/>
         <state_interface name="position">
@@ -40,5 +40,5 @@
         <state_interface name="effort"/>
     </joint>
-    <joint name="joint5">
+    <joint name="${prefix}joint5">
         <command_interface name="position"/>
         <state_interface name="position">
@@ -48,5 +48,5 @@
         <state_interface name="effort"/>
     </joint>
-    <joint name="joint6">
+    <joint name="${prefix}joint6">
         <command_interface name="position"/>
         <state_interface name="position">

File: piper_bringup/urdf/include/mock.ros2_control.xacro (robot description, xacro)
@@ -6,5 +6,5 @@
         <param name="mock_sensor_commands">${mock_sensor_commands}</param>
     </hardware>
-    <joint name="joint1">
+    <joint name="${prefix}joint1">
         <command_interface name="position"/>
         <state_interface name="position">
@@ -14,5 +14,5 @@
         <state_interface name="effort"/>
     </joint>
-    <joint name="joint2">
+    <joint name="${prefix}joint2">
         <command_interface name="position"/>
         <state_interface name="position">
@@ -22,5 +22,5 @@
         <state_interface name="effort"/>
     </joint>
-    <joint name="joint3">
+    <joint name="${prefix}joint3">
         <command_interface name="position"/>
         <state_interface name="position">
@@ -30,5 +30,5 @@
         <state_interface name="effort"/>
     </joint>
-    <joint name="joint4">
+    <joint name="${prefix}joint4">
         <command_interface name="position"/>
         <state_interface name="position">
@@ -38,5 +38,5 @@
         <state_interface name="effort"/>
     </joint>
-    <joint name="joint5">
+    <joint name="${prefix}joint5">
         <command_interface name="position"/>
         <state_interface name="position">
@@ -46,5 +46,5 @@
         <state_interface name="effort"/>
     </joint>
-    <joint name="joint6">
+    <joint name="${prefix}joint6">
         <command_interface name="position"/>
         <state_interface name="position">
